File: quadra-to-ztex/quadra-to-ztex.kicad_pcb (KiCad board)
At the start: 4 copper layers, 100 x 100 mm, 33 parts, among them IC1 74CB3T16211DGGR, IC2 74CB3T16211DGGR, IC3 74CB3T16211DGGR, IC4 74CB3T16211DGGR, J1 Conn_02x07_Odd_Even, J2 10029449-111RLF (HDMI A), J3 A2541HWR-2x6P (Pmod 2x6 F R), U1 TPD12S016PWR, U14 8807-140-170LH

Commit message: fix A18 <-> A19 (hardware)
Connections:
- IC2 pad 22: A29_3V3 -> A28_3V3
- IC2 pad 23: A28_3V3 -> A29_3V3
- JCD1 pad 19: A29_3V3 -> A28_3V3
- JCD1 pad 20: A28_3V3 -> A29_3V3
Routing:
- net A29_3V3: track 50.3 -> 53.0 mm
- net A28_3V3: track 53.0 -> 50.3 mm
